Commit message: more comments

File: assets/ur10e_fixed.urdf (robot description, URDF)
Before this commit: robot ur10e, 13 links, 12 joints
Links:
- link base_link_inertia: geometry collision mesh filename=/home/SIBYL/Dev/pybullet/assets/Universal_Robots/install/ur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; visual mesh filename=/home/SIBYL/Dev/pybullet/assets/Universal_Robots/install/ur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
- link forearm_link: geometry collision mesh filename=/home/SIBYL/Dev/pybullet/assets/Universal_Robots/install/ur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; visual mesh filename=/home/SIBYL/Dev/pybullet/assets/Universal_Robots/install/ur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
- link shoulder_link: geometry collision mesh filename=/home/SIBYL/Dev/pybullet/assets/Universal_Robots/install/ur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; visual mesh filename=/home/SIBYL/Dev/pybullet/assets/Universal_Robots/install/ur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
- link upper_arm_link: geometry collision mesh filename=/home/SIBYL/Dev/pybullet/assets/Universal_Robots/install/ur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; visual mesh filename=/home/SIBYL/Dev/pybullet/assets/Universal_Robots/install/ur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
- link wrist_1_link: geometry collision mesh filename=/home/SIBYL/Dev/pybullet/assets/Universal_Robots/install/ur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; visual mesh filename=/home/SIBYL/Dev/pybullet/assets/Universal_Robots/install/ur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
- link wrist_2_link: geometry collision mesh filename=/home/SIBYL/Dev/pybullet/assets/Universal_Robots/install/ur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; visual mesh filename=/home/SIBYL/Dev/pybullet/assets/Universal_Robots/install/ur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
- link wrist_3_link: geometry collision mesh filename=/home/SIBYL/Dev/pybullet/assets/Universal_Robots/install/ur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; visual mesh filename=/home/SIBYL/Dev/pybullet/assets/Universal_Robots/install/ur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
